Commit message: update

File: src/robot_base/urdf/agrobot.xacro (robot description, xacro)
@@ -38,34 +38,32 @@
     <xacro:property name="M_PI" value="3.14159265359"/>
     <!-- 车体盒子尺寸 -->
-    <xacro:property name="vehicle_length" value="0.650"/>
+    <xacro:property name="vehicle_length" value="0.640"/>
     <!-- x -->
-    <xacro:property name="vehicle_width" value="0.500"/>
+    <xacro:property name="vehicle_width" value="0.542"/>
     <!-- y -->
-    <xacro:property name="vehicle_height" value="0.163"/>
+    <xacro:property name="vehicle_height" value="0.2"/>
     <!-- z -->
-    <!-- 车体离地高度 -->
-    <xacro:property name="ground_clearance" value="0.047"/>
     <!-- 车体中间雷达层尺寸 -->
-     <xacro:property name="middle_length" value="0.498"/>
-     <xacro:property name="middle_width" value="0.348"/>
-     <xacro:property name="middle_height" value="0.066"/>
+    <xacro:property name="middle_length" value="0.498"/>
+    <xacro:property name="middle_width" value="0.348"/>
+    <xacro:property name="middle_height" value="0.066"/>
     <!-- 轮子 -->
     <xacro:property name="wheel_radius" value="0.0875"/>
-    <!-- 170 mm / 2 (原来的两倍) -->
+    <!-- 175 mm / 2 (原来的两倍) -->
     <xacro:property name="wheel_length" value="0.045"/>
-    <xacro:property name="wheel_offset_z" value="${vehicle_height/2 + ground_clearance - wheel_radius}"/>
+    <xacro:property name="wheel_offset_z" value="${wheel_radius + vehicle_height/2}"/>
     <!-- 轮子相对base_link的Z偏移 -->
-    <xacro:property name="wheel_offset_x" value="0"/>
+    <xacro:property name="wheel_offset_x" value="0.236"/>
     <!-- 轮子相对车体中心的X偏移 -->
-    <xacro:property name="wheel_offset_y" value="0.20"/>
+    <xacro:property name="wheel_offset_y" value="0.306"/>
     <!-- 轮子相对车体中心的Y偏移 -->
-    <!-- 实际轮距（两轮中心距离） 0.2*2 = 0.4 -->
+    <!-- 实际轮距（两轮中心距离） 0.306*2 = 0.612 -->
     <xacro:property name="wheel_separation" value="${2 * wheel_offset_y}"/>
     <!-- 万向轮 -->
     <xacro:property name="caster_radius" value="0.0275"/>
     <xacro:property name="caster_length" value="0.045"/>
-    <xacro:property name="caster_offset_z" value="${vehicle_height/2 + ground_clearance - caster_radius}"/>
-    <xacro:property name="caster_offset_y" value="0.18"/>
-    <xacro:property name="caster_offset_x" value="0.25"/>
+    <xacro:property name="caster_offset_z" value="${wheel_radius + vehicle_height/2}"/>
+    <xacro:property name="caster_offset_y" value="0"/>
+    <xacro:property name="caster_offset_x" value="-0.25"/>
     <!-- 单目摄像头：嵌入车体前部内侧，距前表面 20mm，距下表面 224mm -->
     <!-- 摄像头尺寸：长x宽x高 = 50mm x 40mm x 30mm，便于可视化 -->
@@ -242,5 +240,5 @@
         <inertial>
             <mass value="50"/>
-            <inertia ixx="${(1/12)*50*(middle_width*middle_width + middle_height*middle_height)}" ixy="0" ixz="0" iyy="${(1/12)*50*(middle_length*middle_length + middle_height*middle_height)}" iyz="0" izz="${(1/12)*50*(vehicle_length*vehicle_length + vehicle_width*vehicle_width)}"/>
+            <inertia ixx="${(1/12)*50*(middle_width*middle_width + middle_height*middle_height)}" ixy="0" ixz="0" iyy="${(1/12)*50*(middle_length*middle_length + middle_height*middle_height)}" iyz="0" izz="${(1/12)*50*(middle_length*middle_length + middle_width*middle_width)}"/>
         </inertial>
     </link>
@@ -274,15 +272,12 @@
     </joint>
     <!-- ======================== 万向轮 ======================== -->
-    <xacro:caster_link name="rear_l" parent_link="base_link" x_offset_caster="${-caster_offset_x}" y_offset_caster="${caster_offset_y}" z_offset_caster="${-caster_offset_z}"/>
-    <xacro:caster_link name="rear_r" parent_link="base_link" x_offset_caster="${-caster_offset_x}" y_offset_caster="${-caster_offset_y}" z_offset_caster="${-caster_offset_z}"/>
-    <xacro:caster_link name="front" parent_link="base_link" x_offset_caster="${caster_offset_x}" y_offset_caster="0" z_offset_caster="${-caster_offset_z}"/>
-    <!-- ======================== 驱动轮（左右中置） ======================== -->
-    <xacro:wheel_link name="left" parent_link="base_link" x_offset="0" y_offset="${wheel_offset_y}" z_offset="${-wheel_offset_z}"/>
-    <xacro:wheel_link name="right" parent_link="base_link" x_offset="0" y_offset="${-wheel_offset_y}" z_offset="${-wheel_offset_z}"/>
+    <xacro:caster_link name="back" parent_link="base_link" x_offset_caster="${caster_offset_x}" y_offset_caster="${-caster_offset_y}" z_offset_caster="${-caster_offset_z}"/>
+    <!-- ======================== 驱动轮 ======================== -->
+    <xacro:wheel_link name="left" parent_link="base_link" x_offset="${wheel_offset_x}" y_offset="${wheel_offset_y}" z_offset="${-wheel_offset_z}"/>
+    <xacro:wheel_link name="right" parent_link="base_link" x_offset="${wheel_offset_x}" y_offset="${-wheel_offset_y}" z_offset="${-wheel_offset_z}"/>
     <!-- ======================== 摄像头 ======================== -->
     <xacro:camera_link name="right" x_offset_camera="${cam_offset_x}" y_offset_camera="${cam_offset_y}" z_offset_camera="${cam_offset_z}" yaw_offset_camera="${cam_offset_yaw}"/>
     <!-- ======================== 激光雷达 ======================== -->
     <xacro:laser_link name="rightFront" x_offset_laser="${lidar_offset_x}" y_offset_laser="${-lidar_offset_y}" z_offset_laser="${lidar_offset_z}" yaw_offset_laser="${-M_PI/4}"/>
-    <xacro:laser_link name="leftRear" x_offset_laser="${-lidar_offset_x-0.01}" y_offset_laser="${lidar_offset_y-0.01}" z_offset_laser="${lidar_offset_z}" yaw_offset_laser="${3*M_PI/4 - 0.01}"/>
     <!-- ======================== ros2_control 配置 ======================== -->
     <ros2_control name="agrobot" type="system">

Commit message: update

File: src/robot_base/urdf/agrobot.xacro (robot description, xacro)
@@ -44,4 +44,6 @@
     <xacro:property name="vehicle_height" value="0.2"/>
     <!-- z -->
+    <!-- base_link 距离地面的高度：一半车高 + 轮子半径-->
+    <xacro:property name="base_z_origin" value="${wheel_radius + vehicle_height/2}"/>
     <!-- 车体中间雷达层尺寸 -->
     <xacro:property name="middle_length" value="0.498"/>
@@ -52,5 +54,5 @@
     <!-- 175 mm / 2 (原来的两倍) -->
     <xacro:property name="wheel_length" value="0.045"/>
-    <xacro:property name="wheel_offset_z" value="${wheel_radius + vehicle_height/2}"/>
+    <xacro:property name="wheel_offset_z" value="${vehicle_height/2}"/>
     <!-- 轮子相对base_link的Z偏移 -->
     <xacro:property name="wheel_offset_x" value="0.236"/>
@@ -63,5 +65,5 @@
     <xacro:property name="caster_radius" value="0.0275"/>
     <xacro:property name="caster_length" value="0.045"/>
-    <xacro:property name="caster_offset_z" value="${wheel_radius + vehicle_height/2}"/>
+    <xacro:property name="caster_offset_z" value="${base_z_origin - caster_radius}"/>
     <xacro:property name="caster_offset_y" value="0"/>
     <xacro:property name="caster_offset_x" value="-0.25"/>
@@ -202,5 +204,5 @@
         <parent link="base_footprint"/>
         <child link="base_link"/>
-        <origin xyz="0 0 ${wheel_offset_z}" rpy="0 0 0"/>
+        <origin xyz="0 0 ${base_z_origin}" rpy="0 0 0"/>
     </joint>
     <link name="base_link">

Commit message: update xacro

File: src/robot_base/urdf/agrobot.xacro (robot description, xacro)
@@ -1,5 +1,4 @@
 <?xml version="1.0"?>
-<robot name="agrobot"
-    xmlns:xacro="http://www.ros.org/wiki/xacro">
+<robot name="agrobot" xmlns:xacro="http://www.ros.org/wiki/xacro">
     <!-- XACRO参数：可以在launch文件中传递 -->
     <xacro:arg name="controllers_file" default=""/>
@@ -8,40 +7,29 @@
     <xacro:property name="controllers_file" value="$(arg controllers_file)"/>
     <!-- ======================== 常用颜色 ======================== -->
-    <material name="orange">
-        <color rgba="1.0 0.5 0.2 1.0"/>
-    </material>
-    <material name="gray">
-        <color rgba="0.5 0.5 0.5 1.0"/>
-    </material>
-    <material name="dark_gray">
-        <color rgba="0.3 0.3 0.3 1.0"/>
-    </material>
-    <material name="blue">
-        <color rgba="0.2 0.4 0.8 0.5"/>
-    </material>
-    <material name="black">
-        <color rgba="0.1 0.1 0.1 1.0"/>
-    </material>
-    <material name="red">
-        <color rgba="0.8 0.2 0.2 1.0"/>
-    </material>
-    <material name="green">
-        <color rgba="0.2 0.8 0.2 1.0"/>
-    </material>
-    <material name="white">
-        <color rgba="0.9 0.9 0.9 1.0"/>
-    </material>
-    <material name="silver">
-        <color rgba="0.7 0.7 0.7 1.0"/>
-    </material>
+    <material name="orange"><color rgba="1.0 0.5 0.2 1.0"/></material>
+    <material name="gray"><color rgba="0.5 0.5 0.5 1.0"/></material>
+    <material name="dark_gray"><color rgba="0.3 0.3 0.3 1.0"/></material>
+    <material name="blue"><color rgba="0.2 0.4 0.8 0.5"/></material>
+    <material name="black"><color rgba="0.1 0.1 0.1 1.0"/></material>
+    <material name="red"><color rgba="0.8 0.2 0.2 1.0"/></material>
+    <material name="green"><color rgba="0.2 0.8 0.2 1.0"/></material>
+    <material name="white"><color rgba="0.9 0.9 0.9 1.0"/></material>
+    <material name="silver"><color rgba="0.7 0.7 0.7 1.0"/></material>
     <!-- ======================== 几何/安装参数 ======================== -->
     <xacro:property name="M_PI" value="3.14159265359"/>
     <!-- 车体盒子尺寸 -->
-    <xacro:property name="vehicle_length" value="0.640"/>
-    <!-- x -->
-    <xacro:property name="vehicle_width" value="0.542"/>
-    <!-- y -->
-    <xacro:property name="vehicle_height" value="0.2"/>
-    <!-- z -->
+    <xacro:property name="vehicle_length" value="0.640"/> <!-- x -->
+    <xacro:property name="vehicle_width" value="0.542"/>  <!-- y -->
+    <xacro:property name="vehicle_height" value="0.2"/>   <!-- z -->
+    <!-- 轮子 -->
+    <xacro:property name="wheel_radius" value="0.0875"/>
+    <xacro:property name="wheel_length" value="0.045"/>
+    <xacro:property name="wheel_offset_z" value="${vehicle_height/2}"/>
+    <!-- 轮子相对车体中心的X偏移 -->
+    <xacro:property name="wheel_offset_x" value="0.236"/>
+    <xacro:property name="wheel_offset_y" value="0.306"/>
+    <xacro:property name="wheel_separation" value="${2 * wheel_offset_y}"/>
+    <!-- 车体几何中心（外壳）相对于运动学中心（base_link/轮轴）的偏移 -->
+    <xacro:property name="chassis_offset_x" value="${-wheel_offset_x}"/>
     <!-- base_link 距离地面的高度：一半车高 + 轮子半径-->
     <xacro:property name="base_z_origin" value="${wheel_radius + vehicle_height/2}"/>
@@ -50,16 +38,4 @@
     <xacro:property name="middle_width" value="0.348"/>
     <xacro:property name="middle_height" value="0.066"/>
-    <!-- 轮子 -->
-    <xacro:property name="wheel_radius" value="0.0875"/>
-    <!-- 175 mm / 2 (原来的两倍) -->
-    <xacro:property name="wheel_length" value="0.045"/>
-    <xacro:property name="wheel_offset_z" value="${vehicle_height/2}"/>
-    <!-- 轮子相对base_link的Z偏移 -->
-    <xacro:property name="wheel_offset_x" value="0.236"/>
-    <!-- 轮子相对车体中心的X偏移 -->
-    <xacro:property name="wheel_offset_y" value="0.306"/>
-    <!-- 轮子相对车体中心的Y偏移 -->
-    <!-- 实际轮距（两轮中心距离） 0.306*2 = 0.612 -->
-    <xacro:property name="wheel_separation" value="${2 * wheel_offset_y}"/>
     <!-- 万向轮 -->
     <xacro:property name="caster_radius" value="0.0275"/>
@@ -68,6 +44,5 @@
     <xacro:property name="caster_offset_y" value="0"/>
     <xacro:property name="caster_offset_x" value="-0.25"/>
-    <!-- 单目摄像头：嵌入车体前部内侧，距前表面 20mm，距下表面 224mm -->
-    <!-- 摄像头尺寸：长x宽x高 = 50mm x 40mm x 30mm，便于可视化 -->
+    <!-- 单目摄像头 -->
     <xacro:property name="camera_length" value="0.05"/>
     <xacro:property name="camera_width" value="0.05"/>
@@ -77,5 +52,5 @@
     <xacro:property name="cam_offset_z" value="${vehicle_height/2 + middle_height + 0.025}"/>
     <xacro:property name="cam_offset_yaw" value="${M_PI/2}"/>
-    <!-- 激光雷达：嵌入车体顶部前侧，距前表面 5cm，距下表面 15cm -->
+    <!-- 激光雷达 -->
     <xacro:property name="lidar_radius" value="0.032"/>
     <xacro:property name="lidar_length" value="0.05"/>
@@ -154,5 +129,4 @@
             </visual>
             <collision>
-                <origin xyz="0 0 0" rpy="0 0 0"/>
                 <geometry>
                     <cylinder length="${lidar_length}" radius="${lidar_radius}"/>
@@ -160,5 +134,4 @@
             </collision>
             <inertial>
-                <origin xyz="0 0 0" rpy="0 0 0"/>
                 <mass value="0.05"/>
                 <inertia ixx="${0.1*(3*lidar_radius*lidar_radius + lidar_length*lidar_length)/12}" ixy="0" ixz="0" iyy="${0.1*(3*lidar_radius*lidar_radius + lidar_length*lidar_length)/12}" iyz="0" izz="${0.1*lidar_radius*lidar_radius/2}"/>
@@ -166,5 +139,6 @@
         </link>
         <joint name="${name}_laser_joint" type="fixed">
-            <parent link="base_link"/>
+            <!-- 挂载在车体中心 -->
+            <parent link="chassis_link"/>
             <child link="${name}_laser_link"/>
             <origin xyz="${x_offset_laser} ${y_offset_laser} ${z_offset_laser}" rpy="0 0 ${yaw_offset_laser}" />
@@ -173,32 +147,31 @@
     <!-- 摄像头宏 -->
     <xacro:macro name="camera_link" params="name x_offset_camera y_offset_camera z_offset_camera yaw_offset_camera">
-    <link name="${name}_camera">
-        <visual>
-            <origin xyz="0 0 0" rpy="0 0 0"/>
-            <geometry>
-                <box size="${camera_length} ${camera_width} ${camera_height}"/>
-            </geometry>
-            <material name="red"/>
-        </visual>
-        <collision>
-            <origin xyz="0 0 0" rpy="0 0 0"/>
-            <geometry>
-                <box size="${camera_length} ${camera_width} ${camera_height}"/>
-            </geometry>
-        </collision>
-        <inertial>
-            <origin xyz="0 0 0" rpy="0 0 0"/>
-            <mass value="0.05"/>
-            <inertia ixx="${0.05*(camera_width*camera_width + camera_height*camera_height)/12}" ixy="0" ixz="0" iyy="${0.05*(camera_length*camera_length + camera_height*camera_height)/12}" iyz="0" izz="${0.05*(camera_length*camera_length + camera_width*camera_width)/12}"/>
-        </inertial>
-    </link>
-    <joint name="camera_joint" type="fixed">
-        <parent link="base_link"/>
-        <child link="${name}_camera"/>
-        <origin xyz="${x_offset_camera} ${y_offset_camera} ${z_offset_camera}" rpy="0 ${M_PI/2} ${yaw_offset_camera}"/>
-    </joint>
-     </xacro:macro>
-    <!-- ======================== 车体结构 ======================== -->
+        <link name="${name}_camera">
+            <visual>
+                <geometry>
+                    <box size="${camera_length} ${camera_width} ${camera_height}"/>
+                </geometry>
+                <material name="red"/>
+            </visual>
+            <collision>
+                <geometry>
+                    <box size="${camera_length} ${camera_width} ${camera_height}"/>
+                </geometry>
+            </collision>
+            <inertial>
+                <mass value="0.05"/>
+                <inertia ixx="${0.05*(camera_width*camera_width + camera_height*camera_height)/12}" ixy="0" ixz="0" iyy="${0.05*(camera_length*camera_length + camera_height*camera_height)/12}" iyz="0" izz="${0.05*(camera_length*camera_length + camera_width*camera_width)/12}"/>
+            </inertial>
+        </link>
+        <!-- 关节名加上前缀防止重名，挂载在车体中心 -->
+        <joint name="${name}_camera_joint" type="fixed">
+            <parent link="chassis_link"/>
+            <child link="${name}_camera"/>
+            <origin xyz="${x_offset_camera} ${y_offset_camera} ${z_offset_camera}" rpy="0 ${M_PI/2} ${yaw_offset_camera}"/>
+        </joint>
+    </xacro:macro>
+    <!-- ======================== 车体结构 (核心分离部分) ======================== -->
     <link name="base_footprint"/>
+    <!-- 1. base_link: 纯粹的运动学中心，无质量无外观 -->
     <joint name="base_joint" type="fixed">
         <parent link="base_footprint"/>
@@ -206,5 +179,12 @@
         <origin xyz="0 0 ${base_z_origin}" rpy="0 0 0"/>
     </joint>
-    <link name="base_link">
+    <link name="base_link" />
+    <!-- 2. chassis_link: 物理车壳，挂在 base_link 后面 -->
+    <joint name="chassis_joint" type="fixed">
+        <parent link="base_link"/>
+        <child link="chassis_link"/>
+        <origin xyz="${chassis_offset_x} 0 0" rpy="0 0 0"/>
+    </joint>
+    <link name="chassis_link">
         <visual>
             <geometry>
@@ -223,6 +203,7 @@
         </inertial>
     </link>
+    <!-- 中间层，挂在 chassis_link 上 -->
     <joint name="base_middle_joint" type="fixed">
-        <parent link="base_link"/>
+        <parent link="chassis_link"/>
         <child link="base_middle_link"/>
         <origin xyz="0 0 ${vehicle_height/2+middle_height/2}" rpy="0 0 0"/>
@@ -246,19 +227,11 @@
     </link>
     <!-- ======================== IMU传感器 ======================== -->
-    <!-- IMU安装在机器人中心位置，与base_link重合 -->
     <link name="imu_link">
         <visual>
-            <origin xyz="0 0 0" rpy="0 0 0"/>
-            <geometry>
-                <box size="0.02 0.02 0.01"/>
-                <!-- 小盒子表示IMU -->
-            </geometry>
+            <geometry><box size="0.02 0.02 0.01"/></geometry>
             <material name="green"/>
         </visual>
         <collision>
-            <origin xyz="0 0 0" rpy="0 0 0"/>
-            <geometry>
-                <box size="0.02 0.02 0.01"/>
-            </geometry>
+            <geometry><box size="0.02 0.02 0.01"/></geometry>
         </collision>
         <inertial>
@@ -267,15 +240,17 @@
         </inertial>
     </link>
+    <!-- IMU安装在机器人车体物理中心位置，因此挂在 chassis_link -->
     <joint name="imu_joint" type="fixed">
-        <parent link="base_link"/>
+        <parent link="chassis_link"/>
         <child link="imu_link"/>
         <origin xyz="0 0 0" rpy="0 0 0"/>
-        <!-- {{ AURA-X: Fix - IMU安装在base_link中心位置，作为tracking frame. }} -->
     </joint>
     <!-- ======================== 万向轮 ======================== -->
-    <xacro:caster_link name="back" parent_link="base_link" x_offset_caster="${caster_offset_x}" y_offset_caster="${-caster_offset_y}" z_offset_caster="${-caster_offset_z}"/>
+    <!-- 相对车壳测量，挂在 chassis_link -->
+    <xacro:caster_link name="back" parent_link="chassis_link" x_offset_caster="${caster_offset_x}" y_offset_caster="${-caster_offset_y}" z_offset_caster="${-caster_offset_z}"/>
     <!-- ======================== 驱动轮 ======================== -->
-    <xacro:wheel_link name="left" parent_link="base_link" x_offset="${wheel_offset_x}" y_offset="${wheel_offset_y}" z_offset="${-wheel_offset_z}"/>
-    <xacro:wheel_link name="right" parent_link="base_link" x_offset="${wheel_offset_x}" y_offset="${-wheel_offset_y}" z_offset="${-wheel_offset_z}"/>
+    <!-- 挂在 base_link，并且 X_offset 传入 0，使其完美在 base_link 居中！ -->
+    <xacro:wheel_link name="left" parent_link="base_link" x_offset="0" y_offset="${wheel_offset_y}" z_offset="${-wheel_offset_z}"/>
+    <xacro:wheel_link name="right" parent_link="base_link" x_offset="0" y_offset="${-wheel_offset_y}" z_offset="${-wheel_offset_z}"/>
     <!-- ======================== 摄像头 ======================== -->
     <xacro:camera_link name="right" x_offset_camera="${cam_offset_x}" y_offset_camera="${cam_offset_y}" z_offset_camera="${cam_offset_z}" yaw_offset_camera="${cam_offset_yaw}"/>

Commit message: update xacro laser

File: src/robot_base/urdf/agrobot.xacro (robot description, xacro)
@@ -119,5 +119,5 @@
     </xacro:macro>
     <!-- 激光雷达宏 -->
-    <xacro:macro name="laser_link" params="name x_offset_laser y_offset_laser z_offset_laser yaw_offset_laser">
+    <xacro:macro name="laser_link" params="name x_offset_laser y_offset_laser z_offset_laser pitch_offset_laser yaw_offset_laser">
         <link name="${name}_laser_link">
             <visual>
@@ -142,5 +142,5 @@
             <parent link="chassis_link"/>
             <child link="${name}_laser_link"/>
-            <origin xyz="${x_offset_laser} ${y_offset_laser} ${z_offset_laser}" rpy="0 0 ${yaw_offset_laser}" />
+            <origin xyz="${x_offset_laser} ${y_offset_laser} ${z_offset_laser}" rpy="0 ${pitch_offset_laser} ${yaw_offset_laser}" />
         </joint>
     </xacro:macro>
@@ -256,5 +256,5 @@
     <xacro:camera_link name="right" x_offset_camera="${cam_offset_x}" y_offset_camera="${cam_offset_y}" z_offset_camera="${cam_offset_z}" yaw_offset_camera="${cam_offset_yaw}"/>
     <!-- ======================== 激光雷达 ======================== -->
-    <xacro:laser_link name="front" x_offset_laser="${lidar_offset_x}" y_offset_laser="${-lidar_offset_y}" z_offset_laser="${lidar_offset_z}" yaw_offset_laser="${-M_PI/4}"/>
+    <xacro:laser_link name="front" x_offset_laser="${lidar_offset_x}" y_offset_laser="${-lidar_offset_y}" z_offset_laser="${lidar_offset_z}" pitch_offset_laser="${-M_PI/4}" yaw_offset_laser="0"/>
     <!-- ======================== ros2_control 配置 ======================== -->
     <ros2_control name="agrobot" type="system">
