Commit message: update

File: src/robot_base/urdf/agrobot.xacro (robot description, xacro)
@@ -34,8 +34,7 @@
     <!-- base_link 距离地面的高度：一半车高 + 轮子半径-->
     <xacro:property name="base_z_origin" value="${wheel_radius + vehicle_height/2}"/>
-    <!-- 车体中间雷达层尺寸 -->
-    <xacro:property name="middle_length" value="0.498"/>
-    <xacro:property name="middle_width" value="0.348"/>
-    <xacro:property name="middle_height" value="0.066"/>
+    <!-- 车体中间层尺寸 -->
+    <xacro:property name="middle_radius" value="0.300"/>
+    <xacro:property name="middle_height" value="0.21"/>
     <!-- 万向轮 -->
     <xacro:property name="caster_radius" value="0.0275"/>
@@ -53,9 +52,13 @@
     <xacro:property name="cam_offset_yaw" value="${M_PI/2}"/>
     <!-- 激光雷达 -->
-    <xacro:property name="lidar_radius" value="0.032"/>
-    <xacro:property name="lidar_length" value="0.05"/>
-    <xacro:property name="lidar_offset_x" value="0.270"/>
-    <xacro:property name="lidar_offset_y" value="0.200"/>
-    <xacro:property name="lidar_offset_z" value="${vehicle_height/2 + lidar_length/2}"/>
+    <xacro:property name="lidar_radius" value="0.0325"/>
+    <xacro:property name="lidar_length" value="0.06"/>
+    <xacro:property name="lidar_offset_x" value="0.320"/>
+    <xacro:property name="lidar_offset_y" value="0.241"/>
+    <xacro:property name="lidar_offset_z" value="${-vehicle_height/2 + 0.16}"/>
+    <!-- IMU -->
+    <xacro:property name="imu_offset_x" value="0.257"/>
+    <xacro:property name="imu_offset_y" value="0"/>
+    <xacro:property name="imu_offset_z" value="0.03"/>
     <!-- ======================== 通用宏 ======================== -->
     <!-- 轮子宏 -->
@@ -212,5 +215,5 @@
         <visual>
             <geometry>
-                <box size="${middle_length} ${middle_width} ${middle_height}"/>
+                <cylinder radius="${middle_radius}" length="${middle_height}"/>
             </geometry>
             <material name="blue"/>
@@ -218,10 +221,14 @@
         <collision>
             <geometry>
-                <box size="${middle_length} ${middle_width} ${middle_height}"/>
+                <cylinder radius="${middle_radius}" length="${middle_height}"/>
             </geometry>
         </collision>
         <inertial>
             <mass value="50"/>
-            <inertia ixx="${(1/12)*50*(middle_width*middle_width + middle_height*middle_height)}" ixy="0" ixz="0" iyy="${(1/12)*50*(middle_length*middle_length + middle_height*middle_height)}" iyz="0" izz="${(1/12)*50*(middle_length*middle_length + middle_width*middle_width)}"/>
+            <inertia ixx="${(1/12)*50*(3*middle_radius*middle_radius + middle_height*middle_height)}"
+                     ixy="0" ixz="0"
+                     iyy="${(1/12)*50*(3*middle_radius*middle_radius + middle_height*middle_height)}"
+                     iyz="0"
+                     izz="${0.5*50*middle_radius*middle_radius}"/>
         </inertial>
     </link>
@@ -244,5 +251,5 @@
         <parent link="chassis_link"/>
         <child link="imu_link"/>
-        <origin xyz="0 0 0" rpy="0 0 0"/>
+        <origin xyz="${-imu_offset_x} 0 ${-imu_offset_z}" rpy="0 0 0"/>
     </joint>
     <!-- ======================== 万向轮 ======================== -->

Commit message: add pot trans logic to uart

File: src/robot_base/urdf/agrobot.xacro (robot description, xacro)
@@ -285,10 +285,24 @@
         <joint name="right_wheel_joint">
             <command_interface name="velocity">
-                <param name="min">-10.0</param>
-                <param name="max">10.0</param>
+                <param name="min">-1.0</param>
+                <param name="max">1.0</param>
             </command_interface>
             <state_interface name="position"/>
             <state_interface name="velocity"/>
         </joint>
+        <joint name="pot_transfer_joint">
+            <command_interface name="rack_index">
+                <param name="min">-5</param>
+                <param name="max">5</param>
+            </command_interface>
+            <!--  动作类型：0不修改 1搬运 2卸载 3slave -->
+            <command_interface name="action_type"/>
+            <!--  使能触发：0不修改 1使能 2失能 -->
+            <command_interface name="action_enable_cmd"/>
+            <!--  状态反馈：0未进行/已完成 1正在进行 -->
+            <state_interface name="action_running"/>
+            <!--  接管状态：0遥控器未接管 1遥控器强制接管 -->
+            <state_interface name="rc_force_ctl"/>
+        </joint>
     </ros2_control>
 </robot>

Commit message: add pot trans logic to uart

File: src/robot_base/urdf/agrobot.xacro (robot description, xacro)
@@ -291,13 +291,5 @@
             <state_interface name="velocity"/>
         </joint>
-        <joint name="pot_transfer_joint">
-            <command_interface name="rack_index">
-                <param name="min">-5.0</param>
-                <param name="max">5.0</param>
-            </command_interface>
-            <!--  动作类型：0不修改 1搬运 2卸载 3slave -->
-            <command_interface name="action_type"/>
-            <!--  使能触发：0不修改 1使能 2失能 -->
-            <command_interface name="action_enable_cmd"/>
+        <joint name="robot_state_joint">
             <!--  状态反馈：0未进行/已完成 1正在进行 -->
             <state_interface name="action_running"/>

Commit message: add action logic

File: src/robot_base/urdf/agrobot.xacro (robot description, xacro)
@@ -291,10 +291,4 @@
             <state_interface name="velocity"/>
         </joint>
-        <joint name="robot_state_joint">
-            <!--  状态反馈：0未进行/已完成 1正在进行 -->
-            <state_interface name="action_running"/>
-            <!--  接管状态：0遥控器未接管 1遥控器强制接管 -->
-            <state_interface name="rc_force_ctl"/>
-        </joint>
     </ros2_control>
 </robot>
