Commit message: sync: 从 demo 同步源码改动，不含实验脚本和数据
- plant_detector: 新增 PlantMetrics 消息、分段计时、指标发布
- robot_base: 新增 agrobot URDF、更新 EKF 配置、删除旧 launch
- robot_localization: 更新 fastlio2 launch、ICP 参数、EKF 配置
- robot_relocalization: 更新 ICP 配置和实现

Co-Authored-By: Claude Opus 4.7 <noreply@anthropic.com>

File: src/robot_base/urdf/agrobot.xacro (robot description, xacro)
@@ -80,6 +80,6 @@
             <inertial>
                 <origin xyz="0 0 0" rpy="${M_PI/2} 0 0"/>
-                <mass value="0.5"/>
-                <inertia ixx="${0.5*(3*wheel_radius*wheel_radius + wheel_length*wheel_length)/12}" ixy="0" ixz="0" iyy="${0.5*(3*wheel_radius*wheel_radius + wheel_length*wheel_length)/12}" iyz="0" izz="${0.5*wheel_radius*wheel_radius/2}"/>
+                <mass value="5.0"/>
+                <inertia ixx="${5.0*(3*wheel_radius*wheel_radius + wheel_length*wheel_length)/12}" ixy="0" ixz="0" iyy="${5.0*(3*wheel_radius*wheel_radius + wheel_length*wheel_length)/12}" iyz="0" izz="${5.0*wheel_radius*wheel_radius/2}"/>
             </inertial>
         </link>
@@ -89,6 +89,6 @@
             <origin xyz="${x_offset} ${y_offset} ${z_offset}" rpy="0 0 0"/>
             <axis xyz="0 1 0"/>
-            <limit effort="10.0" velocity="10.0"/>
-            <dynamics damping="0.1" friction="0.1"/>
+            <limit effort="10000.0" velocity="1000.0"/>
+            <dynamics damping="0.0" friction="0.0"/>
         </joint>
     </xacro:macro>
@@ -104,13 +104,13 @@
             </visual>
             <collision>
-                <origin xyz="0 0 0" rpy="${M_PI/2} 0 0"/>
-                <geometry>
-                    <cylinder length="${caster_length}" radius="${caster_radius}"/>
-                </geometry>
-            </collision>
-            <inertial>
-                <origin xyz="0 0 0" rpy="${M_PI/2} 0 0"/>
+                <origin xyz="0 0 0" rpy="0 0 0"/>
+                <geometry>
+                    <sphere radius="${caster_radius}"/>
+                </geometry>
+            </collision>
+            <inertial>
+                <origin xyz="0 0 0" rpy="0 0 0"/>
                 <mass value="0.1"/>
-                <inertia ixx="${0.1*(3*caster_radius*caster_radius + caster_length*caster_length)/12}" ixy="0" ixz="0" iyy="${0.1*(3*caster_radius*caster_radius + caster_length*caster_length)/12}" iyz="0" izz="${0.1*caster_radius*caster_radius/2}"/>
+                <inertia ixx="${0.4*0.1*caster_radius*caster_radius}" ixy="0" ixz="0" iyy="${0.4*0.1*caster_radius*caster_radius}" iyz="0" izz="${0.4*0.1*caster_radius*caster_radius}"/>
             </inertial>
         </link>
@@ -202,6 +202,6 @@
         </collision>
         <inertial>
-            <mass value="50"/>
-            <inertia ixx="${(1/12)*50*(vehicle_width*vehicle_width + vehicle_height*vehicle_height)}" ixy="0" ixz="0" iyy="${(1/12)*50*(vehicle_length*vehicle_length + vehicle_height*vehicle_height)}" iyz="0" izz="${(1/12)*50*(vehicle_length*vehicle_length + vehicle_width*vehicle_width)}"/>
+            <mass value="30"/>
+            <inertia ixx="${(1/12)*30*(vehicle_width*vehicle_width + vehicle_height*vehicle_height)}" ixy="0" ixz="0" iyy="${(1/12)*30*(vehicle_length*vehicle_length + vehicle_height*vehicle_height)}" iyz="0" izz="${(1/12)*30*(vehicle_length*vehicle_length + vehicle_width*vehicle_width)}"/>
         </inertial>
     </link>
@@ -225,10 +225,10 @@
         </collision>
         <inertial>
-            <mass value="50"/>
-            <inertia ixx="${(1/12)*50*(3*middle_radius*middle_radius + middle_height*middle_height)}"
+            <mass value="10"/>
+            <inertia ixx="${(1/12)*10*(3*middle_radius*middle_radius + middle_height*middle_height)}"
                      ixy="0" ixz="0"
-                     iyy="${(1/12)*50*(3*middle_radius*middle_radius + middle_height*middle_height)}"
+                     iyy="${(1/12)*10*(3*middle_radius*middle_radius + middle_height*middle_height)}"
                      iyz="0"
-                     izz="${0.5*50*middle_radius*middle_radius}"/>
+                     izz="${0.5*10*middle_radius*middle_radius}"/>
         </inertial>
     </link>
@@ -285,6 +285,6 @@
         <joint name="right_wheel_joint">
             <command_interface name="velocity">
-                <param name="min">-1.0</param>
-                <param name="max">1.0</param>
+                <param name="min">-10.0</param>
+                <param name="max">10.0</param>
             </command_interface>
             <state_interface name="position"/>
