Commit message: fix(agrobot): 修正右轮速度限制并万向轮改为可旋转关节
- 右轮 right_wheel_joint 速度限制从 ±1.0 改为 ±10.0，与左轮一致
- 万向轮 back_caster_joint 从 fixed 改为 continuous (Z轴)，支持自由转向

Co-Authored-By: Claude Opus 4.7 <noreply@anthropic.com>

File: src/robot_base/urdf/agrobot.urdf (robot description, URDF)
Before this commit: robot agrobot, 10 links, 9 joints
Joints:
- joint back_caster_joint: axis (none) -> 0 0 1; type fixed -> continuous

File: src/robot_base/urdf/agrobot.xacro (robot description, xacro)
@@ -115,8 +115,10 @@
             </inertial>
         </link>
-        <joint name="${name}_caster_joint" type="fixed">
+        <joint name="${name}_caster_joint" type="continuous">
             <parent link="${parent_link}"/>
             <child link="${name}_caster_link"/>
             <origin xyz="${x_offset_caster} ${y_offset_caster} ${z_offset_caster}" rpy="0 0 0"/>
+            <axis xyz="0 0 1"/>
+            <dynamics damping="0.1" friction="0.0"/>
         </joint>
     </xacro:macro>
@@ -285,6 +287,6 @@
         <joint name="right_wheel_joint">
             <command_interface name="velocity">
-                <param name="min">-1.0</param>
-                <param name="max">1.0</param>
+                <param name="min">-10.0</param>
+                <param name="max">10.0</param>
             </command_interface>
             <state_interface name="position"/>

Commit message: feat(agrobot): 万向轮增加滚动关节
- 万向轮拆分为转向(yaw, Z轴) + 滚动(wheel, Y轴)两个 continuous joint
- 新增 back_caster_fork_link 作为中间连杆

Co-Authored-By: Claude Opus 4.7 <noreply@anthropic.com>

File: src/robot_base/urdf/agrobot.urdf (robot description, URDF)
Before this commit: robot agrobot, 10 links, 9 joints
Links:
- added link back_caster_fork_link
Joints:
- removed joint back_caster_joint
- added joint back_caster_wheel_joint: type continuous, parent back_caster_fork_link, child back_caster_link, origin xyz=0 0 0 rpy=0 0 0, axis 0 1 0
- added joint back_caster_yaw_joint: type continuous, parent chassis_link, child back_caster_fork_link, origin xyz=-0.25 0 -0.16 rpy=0 0 0, axis 0 0 1

File: src/robot_base/urdf/agrobot.xacro (robot description, xacro)
@@ -93,6 +93,16 @@
         </joint>
     </xacro:macro>
-    <!-- 万向轮宏 -->
+    <!-- 万向轮宏（转向 + 滚动） -->
     <xacro:macro name="caster_link" params="name parent_link x_offset_caster y_offset_caster z_offset_caster">
+        <!-- 转向关节：绕竖直轴(Yaw)自由旋转 -->
+        <link name="${name}_caster_fork_link"/>
+        <joint name="${name}_caster_yaw_joint" type="continuous">
+            <parent link="${parent_link}"/>
+            <child link="${name}_caster_fork_link"/>
+            <origin xyz="${x_offset_caster} ${y_offset_caster} ${z_offset_caster}" rpy="0 0 0"/>
+            <axis xyz="0 0 1"/>
+            <dynamics damping="0.1" friction="0.0"/>
+        </joint>
+        <!-- 滚动关节：轮子绕自身轴心(Y)自由转动 -->
         <link name="${name}_caster_link">
             <visual>
@@ -115,10 +125,10 @@
             </inertial>
         </link>
-        <joint name="${name}_caster_joint" type="continuous">
-            <parent link="${parent_link}"/>
+        <joint name="${name}_caster_wheel_joint" type="continuous">
+            <parent link="${name}_caster_fork_link"/>
             <child link="${name}_caster_link"/>
-            <origin xyz="${x_offset_caster} ${y_offset_caster} ${z_offset_caster}" rpy="0 0 0"/>
-            <axis xyz="0 0 1"/>
-            <dynamics damping="0.1" friction="0.0"/>
+            <origin xyz="0 0 0" rpy="0 0 0"/>
+            <axis xyz="0 1 0"/>
+            <dynamics damping="0.05" friction="0.0"/>
         </joint>
     </xacro:macro>

Commit message: fix(agrobot): base_middle_link 质量从50kg改为10kg并更新惯性张量
Co-Authored-By: Claude Opus 4.7 <noreply@anthropic.com>

File: src/robot_base/urdf/agrobot.urdf (robot description, URDF)
Before this commit: robot agrobot, 11 links, 10 joints
Links:
- link base_middle_link: mass 50 -> 10

File: src/robot_base/urdf/agrobot.xacro (robot description, xacro)
@@ -237,10 +237,10 @@
         </collision>
         <inertial>
-            <mass value="50"/>
-            <inertia ixx="${(1/12)*50*(3*middle_radius*middle_radius + middle_height*middle_height)}"
+            <mass value="10"/>
+            <inertia ixx="${(1/12)*10*(3*middle_radius*middle_radius + middle_height*middle_height)}"
                      ixy="0" ixz="0"
-                     iyy="${(1/12)*50*(3*middle_radius*middle_radius + middle_height*middle_height)}"
+                     iyy="${(1/12)*10*(3*middle_radius*middle_radius + middle_height*middle_height)}"
                      iyz="0"
-                     izz="${0.5*50*middle_radius*middle_radius}"/>
+                     izz="${0.5*10*middle_radius*middle_radius}"/>
         </inertial>
     </link>

Commit message: fix(agrobot): 调整质量和万向轮碰撞模型
- 轮子质量 0.5kg → 5.0kg
- 车体质量 50kg → 30kg
- 万向轮改回 fixed joint，碰撞改为 sphere，惯性改为球体公式

Co-Authored-By: Claude Opus 4.7 <noreply@anthropic.com>

File: src/robot_base/urdf/agrobot.urdf (robot description, URDF)
Before this commit: robot agrobot, 11 links, 10 joints
Links:
- removed link back_caster_fork_link
- link back_caster_link: geometry collision sphere radius=0.0275; visual cylinder length=0.045 radius=0.0275
- link chassis_link: mass 50 -> 30
- link left_wheel_link: mass 0.5 -> 5.0
- link right_wheel_link: mass 0.5 -> 5.0
Joints:
- removed joint back_caster_wheel_joint
- removed joint back_caster_yaw_joint
- added joint back_caster_joint: type fixed, parent chassis_link, child back_caster_link, origin xyz=-0.25 0 -0.16 rpy=0 0 0

File: src/robot_base/urdf/agrobot.xacro (robot description, xacro)
@@ -80,6 +80,6 @@
             <inertial>
                 <origin xyz="0 0 0" rpy="${M_PI/2} 0 0"/>
-                <mass value="0.5"/>
-                <inertia ixx="${0.5*(3*wheel_radius*wheel_radius + wheel_length*wheel_length)/12}" ixy="0" ixz="0" iyy="${0.5*(3*wheel_radius*wheel_radius + wheel_length*wheel_length)/12}" iyz="0" izz="${0.5*wheel_radius*wheel_radius/2}"/>
+                <mass value="5.0"/>
+                <inertia ixx="${5.0*(3*wheel_radius*wheel_radius + wheel_length*wheel_length)/12}" ixy="0" ixz="0" iyy="${5.0*(3*wheel_radius*wheel_radius + wheel_length*wheel_length)/12}" iyz="0" izz="${5.0*wheel_radius*wheel_radius/2}"/>
             </inertial>
         </link>
@@ -93,42 +93,30 @@
         </joint>
     </xacro:macro>
-    <!-- 万向轮宏（转向 + 滚动） -->
+    <!-- 万向轮宏 -->
     <xacro:macro name="caster_link" params="name parent_link x_offset_caster y_offset_caster z_offset_caster">
-        <!-- 转向关节：绕竖直轴(Yaw)自由旋转 -->
-        <link name="${name}_caster_fork_link"/>
-        <joint name="${name}_caster_yaw_joint" type="continuous">
+        <link name="${name}_caster_link">
+            <visual>
+                <origin xyz="0 0 0" rpy="${M_PI/2} 0 0"/>
+                <geometry>
+                    <cylinder length="${caster_length}" radius="${caster_radius}"/>
+                </geometry>
+                <material name="gray"/>
+            </visual>
+            <collision>
+                <origin xyz="0 0 0" rpy="0 0 0"/>
+                <geometry>
+                    <sphere radius="${caster_radius}"/>
+                </geometry>
+            </collision>
+            <inertial>
+                <origin xyz="0 0 0" rpy="0 0 0"/>
+                <mass value="0.1"/>
+                <inertia ixx="${0.4*0.1*caster_radius*caster_radius}" ixy="0" ixz="0" iyy="${0.4*0.1*caster_radius*caster_radius}" iyz="0" izz="${0.4*0.1*caster_radius*caster_radius}"/>
+            </inertial>
+        </link>
+        <joint name="${name}_caster_joint" type="fixed">
             <parent link="${parent_link}"/>
-            <child link="${name}_caster_fork_link"/>
+            <child link="${name}_caster_link"/>
             <origin xyz="${x_offset_caster} ${y_offset_caster} ${z_offset_caster}" rpy="0 0 0"/>
-            <axis xyz="0 0 1"/>
-            <dynamics damping="0.1" friction="0.0"/>
-        </joint>
-        <!-- 滚动关节：轮子绕自身轴心(Y)自由转动 -->
-        <link name="${name}_caster_link">
-            <visual>
-                <origin xyz="0 0 0" rpy="${M_PI/2} 0 0"/>
-                <geometry>
-                    <cylinder length="${caster_length}" radius="${caster_radius}"/>
-                </geometry>
-                <material name="gray"/>
-            </visual>
-            <collision>
-                <origin xyz="0 0 0" rpy="${M_PI/2} 0 0"/>
-                <geometry>
-                    <cylinder length="${caster_length}" radius="${caster_radius}"/>
-                </geometry>
-            </collision>
-            <inertial>
-                <origin xyz="0 0 0" rpy="${M_PI/2} 0 0"/>
-                <mass value="0.1"/>
-                <inertia ixx="${0.1*(3*caster_radius*caster_radius + caster_length*caster_length)/12}" ixy="0" ixz="0" iyy="${0.1*(3*caster_radius*caster_radius + caster_length*caster_length)/12}" iyz="0" izz="${0.1*caster_radius*caster_radius/2}"/>
-            </inertial>
-        </link>
-        <joint name="${name}_caster_wheel_joint" type="continuous">
-            <parent link="${name}_caster_fork_link"/>
-            <child link="${name}_caster_link"/>
-            <origin xyz="0 0 0" rpy="0 0 0"/>
-            <axis xyz="0 1 0"/>
-            <dynamics damping="0.05" friction="0.0"/>
         </joint>
     </xacro:macro>
@@ -214,6 +202,6 @@
         </collision>
         <inertial>
-            <mass value="50"/>
-            <inertia ixx="${(1/12)*50*(vehicle_width*vehicle_width + vehicle_height*vehicle_height)}" ixy="0" ixz="0" iyy="${(1/12)*50*(vehicle_length*vehicle_length + vehicle_height*vehicle_height)}" iyz="0" izz="${(1/12)*50*(vehicle_length*vehicle_length + vehicle_width*vehicle_width)}"/>
+            <mass value="30"/>
+            <inertia ixx="${(1/12)*30*(vehicle_width*vehicle_width + vehicle_height*vehicle_height)}" ixy="0" ixz="0" iyy="${(1/12)*30*(vehicle_length*vehicle_length + vehicle_height*vehicle_height)}" iyz="0" izz="${(1/12)*30*(vehicle_length*vehicle_length + vehicle_width*vehicle_width)}"/>
         </inertial>
     </link>

Commit message: fix(agrobot): 轮子关节去掉阻尼摩擦，提高速度和力矩上限
- effort 10 → 10000, velocity 10 → 1000
- damping/friction 0.1 → 0.0

Co-Authored-By: Claude Opus 4.7 <noreply@anthropic.com>

File: src/robot_base/urdf/agrobot.urdf (robot description, URDF)
Before this commit: robot agrobot, 10 links, 9 joints
Joints:
- joint left_wheel_joint: limit effort=10.0 velocity=10.0 -> effort=10000.0 velocity=1000.0
- joint right_wheel_joint: limit effort=10.0 velocity=10.0 -> effort=10000.0 velocity=1000.0

File: src/robot_base/urdf/agrobot.xacro (robot description, xacro)
@@ -89,6 +89,6 @@
             <origin xyz="${x_offset} ${y_offset} ${z_offset}" rpy="0 0 0"/>
             <axis xyz="0 1 0"/>
-            <limit effort="10.0" velocity="10.0"/>
-            <dynamics damping="0.1" friction="0.1"/>
+            <limit effort="10000.0" velocity="1000.0"/>
+            <dynamics damping="0.0" friction="0.0"/>
         </joint>
     </xacro:macro>
